File: CircuitBrains Basic/v1_2/CircuitBrains Basic v1_2/CircuitBrains Basic v1_2.kicad_pcb (KiCad board)
At the start: 2 copper layers, 25 x 25 mm, 23 parts, among them SW1 KMR231, U1 W25Q32JVZPIQ, U2 AP2112K-3.3, U3 ATSAMD21E18A-MU, U4 28SOM

Commit message: Updated docs & updated CB Basic board file to kicad 6 format
Connections:
- net /D1_TX renamed /D1
- U2 pad 4: Net-(U2-Pad4) -> (no net)
Other:
- net class Default removed
